File: bluebird.kicad_pcb (KiCad board)
At the start: 2 copper layers, 310.8 x 126.6 mm, 216 parts, among them J1 USB_C_Receptacle_USB2.0, J2 Conn_01x02_Male, J3 Conn_01x05, SW1 SW_PUSH, U1 ATMEGA32U4, U2 MCP23017_SS, U3 IS31FL3731-SA, U4 PAM2401, U5 MCP73831-2-OT, Y1 FA328 16MHz

Commit message: Attempt to wire LEDs
Routing:
- net LED_CB8: track 99.6 -> 290.3 mm, vias 0 -> 4
- net LED_CB7: track 117.8 -> 234.7 mm, vias 1 -> 3
- net LED_CB6: track 181.3 -> 185.7 mm, vias 1 -> 2
Changed lines of the file:
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@@
     (thickness 1.6)
     (drawings 17)
-    (tracks 2699)
+    (tracks 2729)
     (zones 0)
     (modules 216)
@@
     (pad_to_mask_clearance 0)
     (aux_axis_origin 0 0)
-    (visible_elements 7FFFFFFF)
+    (visible_elements 7FFFF7FF)
     (pcbplotparams
       (layerselection 0x010fc_ffffffff)
@@
       (outputformat 1)
       (mirror false)
-      (drillshape 1)
+      (drillshape 0)
       (scaleselection 1)
       (outputdirectory ""))
@@
   (segment (start 308.718001 39.215399) (end 307.268993 37.766391) (width 1) (layer F.Cu) (net 151))
   (segment (start 322.133 69.3014) (end 322.133 67.954362) (width 1) (layer F.Cu) (net 151))
+  (via (at 285.75 53.594) (size 0.8) (drill 0.4) (layers F.Cu B.Cu) (net 151))
+  (segment (start 284.033 50.2514) (end 284.033 51.877) (width 0.25) (layer F.Cu) (net 151))
+  (segment (start 284.033 51.877) (end 285.75 53.594) (width 0.25) (layer F.Cu) (net 151))
+  (segment (start 285.75 53.594) (end 203.2 53.594) (width 0.25) (layer B.Cu) (net 151))
+  (via (at 181.864 53.594) (size 0.8) (drill 0.4) (layers F.Cu B.Cu) (net 151))
+  (segment (start 203.2 53.594) (end 181.864 53.594) (width 0.25) (layer B.Cu) (net 151))
+  (segment (start 181.864 53.594) (end 179.902999 55.555001) (width 0.25) (layer F.Cu) (net 151))
+  (segment (start 179.902999 69.681401) (end 180.833598 70.612) (width 0.25) (layer F.Cu) (net 151))
+  (segment (start 179.902999 55.555001) (end 179.902999 69.681401) (width 0.25) (layer F.Cu) (net 151))
+  (segment (start 180.833598 70.612) (end 184.658 70.612) (width 0.25) (layer F.Cu) (net 151))
+  (segment (start 193.297999 79.251999) (end 193.297999 100.580001) (width 0.25) (layer F.Cu) (net 151))
+  (segment (start 184.658 70.612) (end 193.297999 79.251999) (width 0.25) (layer F.Cu) (net 151))
+  (via (at 191.008 113.538) (size 0.8) (drill 0.4) (layers F.Cu B.Cu) (net 151))
+  (segment (start 193.297999 100.580001) (end 193.297999 111.248001) (width 0.25) (layer F.Cu) (net 151))
+  (segment (start 193.297999 111.248001) (end 191.008 113.538) (width 0.25) (layer F.Cu) (net 151))
+  (segment (start 188.535499 123.376501) (end 188.468 123.444) (width 0.25) (layer B.Cu) (net 151))
+  (via (at 188.468 123.444) (size 0.8) (drill 0.4) (layers F.Cu B.Cu) (net 151))
+  (segment (start 191.008 113.538) (end 188.535499 116.010501) (width 0.25) (layer B.Cu) (net 151))
+  (segment (start 188.535499 116.010501) (end 188.535499 123.376501) (width 0.25) (layer B.Cu) (net 151))
+  (segment (start 188.468 123.444) (end 188.468 125.73) (width 0.25) (layer F.Cu) (net 151))
   (segment (start 322.133 108.748438) (end 322.133 107.4014) (width 1) (layer F.Cu) (net 152))
   (segment (start 326.096901 119.645989) (end 322.133 115.682088) (width 1) (layer F.Cu) (net 152))
@@
   (segment (start 295.367901 67.648899) (end 293.863463 67.648899) (width 1) (layer F.Cu) (net 152))
   (segment (start 299.193001 62.350599) (end 297.521901 64.021699) (width 1) (layer F.Cu) (net 152))
-  (segment (start 299.193001 51.437307) (end 299.193001 62.350599) (width 1) (layer F.Cu) (net 152))
   (segment (start 298.704 50.948306) (end 299.193001 51.437307) (width 1) (layer F.Cu) (net 152))
   (segment (start 298.704 50.2412) (end 298.704 50.948306) (width 1) (layer F.Cu) (net 152))
+  (via (at 286.512 54.356) (size 0.8) (drill 0.4) (layers F.Cu B.Cu) (net 152))
+  (segment (start 286.530999 54.374999) (end 286.512 54.356) (width 0.25) (layer F.Cu) (net 152))
+  (segment (start 299.193001 54.374999) (end 286.530999 54.374999) (width 0.25) (layer F.Cu) (net 152))
+  (segment (start 299.193001 54.374999) (end 299.193001 62.350599) (width 1) (layer F.Cu) (net 152))
+  (segment (start 299.193001 51.437307) (end 299.193001 54.374999) (width 1) (layer F.Cu) (net 152))
+  (via (at 182.297999 54.494915) (size 0.8) (drill 0.4) (layers F.Cu B.Cu) (net 152))
+  (segment (start 286.512 54.356) (end 182.436914 54.356) (width 0.25) (layer B.Cu) (net 152))
+  (segment (start 182.436914 54.356) (end 182.297999 54.494915) (width 0.25) (layer B.Cu) (net 152))
   (segment (start 265.288463 67.648899) (end 264.983 67.954362) (width 1) (layer F.Cu) (net 153))
   (segment (start 267.935901 67.648899) (end 265.288463 67.648899) (width 1) (layer F.Cu) (net 153))
@@
   (segment (start 307.328829 122.946401) (end 307.046901 122.664473) (width 1) (layer F.Cu) (net 153))
   (segment (start 317.5 129.6924) (end 317.5 124.108398) (width 1) (layer F.Cu) (net 153))
+  (via (at 260.858 50.8) (size 0.8) (drill 0.4) (layers F.Cu B.Cu) (net 153))
+  (segment (start 264.983 50.2514) (end 261.4066 50.2514) (width 0.25) (layer B.Cu) (net 153))
+  (segment (start 261.4066 50.2514) (end 260.858 50.8) (width 0.25) (layer B.Cu) (net 153))
   (segment (start 245.933 67.954362) (end 245.933 69.3014) (width 1) (layer F.Cu) (net 154))
   (segment (start 248.073101 67.648899) (end 246.238463 67.648899) (width 1) (layer F.Cu) (net 154))

Commit message: Ripup all traces, rewire schematic matrix to better fit pcb layout
Routing:
- net LED_CA6: track 476.1 -> 0.00 mm
- net LED_CB1: track 443.7 -> 0.00 mm, vias 2 -> 0
- net col9: track 408.9 -> 0.00 mm, vias 1 -> 0
- net col8: track 393.9 -> 0.00 mm, vias 2 -> 0
- net col12: track 349.0 -> 0.00 mm, vias 2 -> 0
- net LED_CB2: track 339.7 -> 0.00 mm, vias 1 -> 0
- net col13: track 337.7 -> 0.00 mm, vias 1 -> 0
- net col14: track 330.2 -> 0.00 mm, vias 5 -> 0
- net col15: track 324.5 -> 0.00 mm, vias 3 -> 0
- net USB_DP: track 307.1 -> 0.00 mm, vias 2 -> 0
- net LED_CA5: track 302.9 -> 0.00 mm
- net USB_DM: track 302.2 -> 0.00 mm, vias 2 -> 0
- net row0: track 297.8 -> 0.00 mm
- net col7: track 297.5 -> 0.00 mm, vias 3 -> 0
- net row2: track 297.0 -> 0.00 mm
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